Commit message: fix(xr): Phase B5 follow-up — left thumb 미동작 (DG-5F hardware sign convention 발견)
증상 (사용자 실측 2026-05-27):
- left DG-5F 4 finger (index/middle/ring/pinky) 굴곡 OK
- **엄지만 안 굽힘**

근본 원인:
- DG-5F hardware 는 좌/우 동일 단일 motor unit + 동일 회전 convention.
- `dg5f_ros2_client.py` / `dg5f_driver` / `dg5f_*_pid_all_controller.yaml`
  모두 per-joint sign 변환 없음 — radian 값 그대로 motor.
- native `dg5f_left.urdf` 의 sign mirror 는 sim/RViz visualization 전용 —
  실 hardware Modbus 와 mismatch.
- 결정적 증거: native URDF 의 `_*_2` MCP flex joint (axis "0 1 0") 가
  **양쪽 동일 `[0, 2.0]`** — single-sign joint 만 일부 mirror, 양방향 joint
  는 hardware convention 통일 → mirror 가 일관되지 않음.
- `lj_dg_1_2` 는 single-sign (negative-only) joint 라 mirror 시 sign 완전
  반전 — retargeter 가 양수만 출력 → motor 가 반대 방향으로 → thumb 안 굽힘.

수정 (`sender/hand/config_xr/dg5f_left_retarget.urdf`):

4 개 single-sign joint limit 를 right URDF 와 동일하게 변경:

| joint | native (sim) | B5 fix |
|---|---|---|
| lj_dg_1_1 (thumb abd) | [-0.89, 0.38] | [-0.38, 0.89] |
| lj_dg_1_2 (thumb opp) | [0, π]         | [-π, 0]  ⭐ 직접 원인 |
| lj_dg_5_1 (pinky abd) | [-1.05, 0.02] | [-0.02, 1.05] |
| lj_dg_5_2 (pinky flex) | [-0.61, 0.42] | [-0.42, 0.61] |

PIP/DIP (`_*_3`, `_*_4`) 와 MCP flex (`_*_2`) 는 이미 양쪽 동일 — 수정 불요.

검증:
- selftest --hand right: PASS, q20 range [-0.479, 1.048] (negative thumb opp)
- selftest --hand left:  PASS, q20 range [-0.385, 0.502] (negative thumb opp,
  fix 전: [-1.048, 0.477] 의 mirror sign 패턴 — 이제 right 와 동일 패턴)

docs/vr_teleop/xr_spike/B5_left_hand.md: §1.C 새 단락 + 트러블슈팅 표 항목 추가.

다음: 사용자 실 left DG-5F 재테스트 — open / fist / pinch / thumb 모두 동작 확인.

File: sender/hand/config_xr/dg5f_left_retarget.urdf (robot description, URDF)
Before this commit: robot dg5f_left, 28 links, 27 joints
Joints:
- joint lj_dg_1_1: limit lower=-0.8901179185171081 upper=0.3839724354387525 effort=7.5 velocity=3.141592653589793 -> lower=-0.3839724354387525 upper=0.8901179185171081 effort=7.5 velocity=3.141592653589793
- joint lj_dg_1_2: limit lower=-0.0 upper=3.141592653589793 effort=7.5 velocity=3.141592653589793 -> lower=-3.141592653589793 upper=0.0 effort=7.5 velocity=3.141592653589793
- joint lj_dg_2_1: limit lower=-0.6108652381980153 upper=0.4188790204786391 effort=7.5 velocity=3.141592653589793 -> lower=-0.4188790204786391 upper=0.6108652381980153 effort=7.5 velocity=3.141592653589793
- joint lj_dg_5_1: limit lower=-1.0471975511965976 upper=0.017453292519943295 effort=7.5 velocity=3.141592653589793 -> lower=-0.017453292519943295 upper=1.0471975511965976 effort=7.5 velocity=3.141592653589793
- joint lj_dg_5_2: limit lower=-0.6108652381980153 upper=0.4188790204786391 effort=7.5 velocity=3.141592653589793 -> lower=-0.4188790204786391 upper=0.6108652381980153 effort=7.5 velocity=3.141592653589793

Commit message: fix(xr): Phase B5 — 4 sign limit fix revert (사용자 2차 실측 반박)
이전 commit (6d92185) 의 4 개 single-sign joint limit 변경을 revert.

사용자 2차 실측 (2026-05-27):
- "새끼손가락은 이전 (mirror) 이 더 맞음" → mirror sign hardware 일치 확인
- "엄지는 지금 전혀 안 움직임 (수정 전엔 조금이라도 움직였음)" → limit 가 아닌 다른 원인

→ 1차 가설 (hardware 좌/우 동일 회전 convention) 오답.
   실제로는 DG-5F left hardware 도 진짜 mirror motor 회전.
   native dg5f_left.urdf 의 limit 값 hardware 와 일치.

Revert 적용:
- lj_dg_1_1: [-0.38, 0.89] → [-0.89, 0.38] (native)
- lj_dg_1_2: [-π, 0]      → [0, π]         (native)
- lj_dg_5_1: [-0.02, 1.05] → [-1.05, 0.02] (native)
- lj_dg_5_2: [-0.42, 0.61] → [-0.61, 0.42] (native)

selftest --hand left: PASS, range [-1.048, 0.478] (native mirror 패턴).

엄지 미동작 별도 진단:
- limit 와 무관. 가장 가능성 높은 원인:
  MEDIAPIPE_OPERATOR2MANO_LEFT 매트릭스 (mano_transform.py:95-97 의
  "not yet hardware-verified" 경고) 의 chirality 정확성.
- 다음 시도 권장:
  python3 -m sender.hand.xr_hand_sender --hand left --convention manus
  → MANUS_OPERATOR2MANO_LEFT 는 row 1 sign flip 만 다름.

docs/vr_teleop/xr_spike/B5_left_hand.md §1.C 갱신:
- 1차 가설 + 사용자 반박 + revert 기록
- 엄지 미해결 별도 진단 권장 (convention manus toggle / B6 후속)
- 트러블슈팅 표 항목 정정

File: sender/hand/config_xr/dg5f_left_retarget.urdf (robot description, URDF)
Before this commit: robot dg5f_left, 28 links, 27 joints
Joints:
- joint lj_dg_1_1: limit lower=-0.3839724354387525 upper=0.8901179185171081 effort=7.5 velocity=3.141592653589793 -> lower=-0.8901179185171081 upper=0.3839724354387525 effort=7.5 velocity=3.141592653589793
- joint lj_dg_1_2: limit lower=-3.141592653589793 upper=0.0 effort=7.5 velocity=3.141592653589793 -> lower=-0.0 upper=3.141592653589793 effort=7.5 velocity=3.141592653589793
- joint lj_dg_2_1: limit lower=-0.4188790204786391 upper=0.6108652381980153 effort=7.5 velocity=3.141592653589793 -> lower=-0.6108652381980153 upper=0.4188790204786391 effort=7.5 velocity=3.141592653589793
- joint lj_dg_4_1: limit lower=-0.4188790204786391 upper=0.6108652381980153 effort=7.5 velocity=3.141592653589793 -> lower=-0.6108652381980153 upper=0.4188790204786391 effort=7.5 velocity=3.141592653589793
- joint lj_dg_5_1: limit lower=-0.017453292519943295 upper=1.0471975511965976 effort=7.5 velocity=3.141592653589793 -> lower=-1.0471975511965976 upper=0.017453292519943295 effort=7.5 velocity=3.141592653589793
- joint lj_dg_5_2: limit lower=-0.4188790204786391 upper=0.6108652381980153 effort=7.5 velocity=3.141592653589793 -> lower=-0.6108652381980153 upper=0.4188790204786391 effort=7.5 velocity=3.141592653589793

Commit message: fix(xr): Phase B5 final — dg5f_left URDF 출처를 tesollodelto/tesollo_model 로 교체
사용자 3차 실측 (2026-05-27):
- dg5f_ros2 의 dg5f_left.urdf 가 hardware envelope 부정확 — 엄지 안 굽힘.
- [tesollodelto/tesollo_model dg5f_left.urdf](https://github.com/tesollodelto/tesollo_model/blob/main/dg5f/dg5f_left.urdf)
  로 교체하니 hardware 정상 동작 확인 (엄지 포함 모든 손가락).

핵심 차이 (key joint limit):
- lj_dg_1_1 (thumb abd): [-1.34, 0.38] vs dg5f_ros2 의 [-0.89, 0.38]
- lj_dg_1_2 (thumb opp): [0, 2.71] vs dg5f_ros2 의 [0, π]
- lj_dg_5_2: [-π/2, 0.262] vs dg5f_ros2 의 [-0.61, 0.42]

이전 우리 modification 모두 원복 (새 URDF 그대로):
- PIP/DIP `lower=0` modification 제거 (B5 first commit 96e3ee1) — 새 URDF
  의 native [-π/2, π/2] 양방향 그대로 보존.
- 4 single-sign joint sign flip 시도 이미 c31cad2 에서 revert 완료.

수정 (mesh path 만):
- 새 URDF mesh path: `package://meshes/dg5f_left/ll_dg_*.{dae,STL}`
- 우리 폴더 구조에 맞춰: `.dae` → `./meshes/visual/`, `.STL` → `./meshes/collision/`
- meshes 자체는 dg5f_ros2 의 ll_dg_* 그대로 사용 (이름 동일 → 호환).

검증:
- selftest --hand left:  PASS, range [-1.048, 0.476]
- selftest --hand right: PASS, range [-0.479, 1.048]  (회귀 없음)

docs/vr_teleop/xr_spike/B5_left_hand.md §1 갱신:
- B5 진행 단계 4 차례 변경 이력 표 (96e3ee1 → 6d92185 → c31cad2 → final)
- key joint limit 비교표 (tesollodelto vs dg5f_ros2)
- 트러블슈팅 표의 thumb 미해결 항목 → "B5 final 에서 해결됨" 으로 업데이트

File: sender/hand/config_xr/dg5f_left_retarget.urdf (robot description, URDF)
Before this commit: robot dg5f_left, 28 links, 27 joints
Links:
- link ll_dg_1_1: mass 0.045 -> 0.0482
- link ll_dg_1_2: mass 0.025 -> 0.0164
- link ll_dg_1_3: mass 0.045 -> 0.0362
- link ll_dg_1_4: mass 0.045 -> 0.0505
- link ll_dg_2_1: mass 0.045 -> 0.0546
- link ll_dg_2_2: mass 0.045 -> 0.0362
- link ll_dg_2_3: mass 0.045 -> 0.0362
- link ll_dg_2_4: mass 0.025 -> 0.0266
- link ll_dg_3_1: mass 0.045 -> 0.0526
- link ll_dg_3_2: mass 0.045 -> 0.0362
- link ll_dg_3_3: mass 0.045 -> 0.0362
- link ll_dg_3_4: mass 0.025 -> 0.0266
- link ll_dg_4_1: mass 0.045 -> 0.0548
- link ll_dg_4_2: mass 0.045 -> 0.0362
- link ll_dg_4_3: mass 0.045 -> 0.0362
- link ll_dg_4_4: mass 0.025 -> 0.0266
- link ll_dg_5_1: mass 0.055 -> 0.0744
- link ll_dg_5_2: mass 0.025 -> 0.0164
- link ll_dg_5_3: mass 0.045 -> 0.0362
- link ll_dg_5_4: mass 0.045 -> 0.0505
- link ll_dg_base: mass 0.45 -> 0.3529
- link ll_dg_palm: mass 0.35 -> 0.5578
Joints:
- joint lj_dg_1_1: limit lower=-0.8901179185171081 upper=0.3839724354387525 effort=7.5 velocity=3.141592653589793 -> lower=-1.3439035240356338 upper=0.3839724354387525 effort=7.5 velocity=3.141592653589793
- joint lj_dg_1_2: limit lower=-0.0 upper=3.141592653589793 effort=7.5 velocity=3.141592653589793 -> lower=-0.0 upper=2.705260340591211 effort=7.5 velocity=3.141592653589793
- joint lj_dg_1_3: limit lower=0.0 upper=1.5707963267948966 effort=7.5 velocity=3.141592653589793 -> lower=-1.5707963267948966 upper=1.5707963267948966 effort=7.5 velocity=3.141592653589793
- joint lj_dg_1_4: limit lower=0.0 upper=1.5707963267948966 effort=7.5 velocity=3.141592653589793 -> lower=-1.5707963267948966 upper=1.5707963267948966 effort=7.5 velocity=3.141592653589793
- joint lj_dg_2_1: limit lower=-0.6108652381980153 upper=0.4188790204786391 effort=7.5 velocity=3.141592653589793 -> lower=-0.3490658503988659 upper=0.5410520681182421 effort=7.5 velocity=3.141592653589793
- joint lj_dg_2_3: limit lower=0.0 upper=1.5707963267948966 effort=7.5 velocity=3.141592653589793 -> lower=-1.5707963267948966 upper=1.5707963267948966 effort=7.5 velocity=3.141592653589793
- joint lj_dg_2_4: limit lower=0.0 upper=1.5707963267948966 effort=7.5 velocity=3.141592653589793 -> lower=-1.5707963267948966 upper=1.5707963267948966 effort=7.5 velocity=3.141592653589793
- joint lj_dg_3_1: limit lower=-0.6108652381980153 upper=0.6108652381980153 effort=7.5 velocity=3.141592653589793 -> lower=-0.4363323129985824 upper=0.4363323129985824 effort=7.5 velocity=3.141592653589793
- joint lj_dg_3_2: limit lower=0.0 upper=1.9547687622336491 effort=7.5 velocity=3.141592653589793 -> lower=0.0 upper=2.007128639793479 effort=7.5 velocity=3.141592653589793
- joint lj_dg_3_3: limit lower=0.0 upper=1.5707963267948966 effort=7.5 velocity=3.141592653589793 -> lower=-1.5707963267948966 upper=1.5707963267948966 effort=7.5 velocity=3.141592653589793
- joint lj_dg_3_4: limit lower=0.0 upper=1.5707963267948966 effort=7.5 velocity=3.141592653589793 -> lower=-1.5707963267948966 upper=1.5707963267948966 effort=7.5 velocity=3.141592653589793
- joint lj_dg_4_1: limit lower=-0.6108652381980153 upper=0.4188790204786391 effort=7.5 velocity=3.141592653589793 -> lower=-0.5585053606381855 upper=0.2617993877991494 effort=7.5 velocity=3.141592653589793
- joint lj_dg_4_2: limit lower=0.0 upper=1.9024088846738192 effort=7.5 velocity=3.141592653589793 -> lower=0.0 upper=1.9198621771937625 effort=7.5 velocity=3.141592653589793
- joint lj_dg_4_3: limit lower=0.0 upper=1.5707963267948966 effort=7.5 velocity=3.141592653589793 -> lower=-1.5707963267948966 upper=1.5707963267948966 effort=7.5 velocity=3.141592653589793
- joint lj_dg_4_4: limit lower=0.0 upper=1.5707963267948966 effort=7.5 velocity=3.141592653589793 -> lower=-1.5707963267948966 upper=1.5707963267948966 effort=7.5 velocity=3.141592653589793
- joint lj_dg_5_1: limit lower=-1.0471975511965976 upper=0.017453292519943295 effort=7.5 velocity=3.141592653589793 -> lower=-1.0471975511965976 upper=0.0 effort=7.5 velocity=3.141592653589793
- joint lj_dg_5_2: limit lower=-0.6108652381980153 upper=0.4188790204786391 effort=7.5 velocity=3.141592653589793 -> lower=-1.5707963267948966 upper=0.2617993877991494 effort=7.5 velocity=3.141592653589793
- joint lj_dg_5_3: limit lower=0.0 upper=1.5707963267948966 effort=7.5 velocity=3.141592653589793 -> lower=-1.5707963267948966 upper=1.5707963267948966 effort=7.5 velocity=3.141592653589793
- joint lj_dg_5_4: limit lower=0.0 upper=1.5707963267948966 effort=7.5 velocity=3.141592653589793 -> lower=-1.5707963267948966 upper=1.5707963267948966 effort=7.5 velocity=3.141592653589793
